Commit message: Primo test funzionante

File: lwr_testing/sensors/asus_camera.urdf.xacro (robot description, xacro)
@@ -35,5 +35,6 @@
       </link>
       <joint name="${name}_depth_joint" type="fixed">
-        <origin xyz="0.0 0.049 0.0" rpy="0 0 0" />
+        <!--<origin xyz="0.0 0.049 0.0" rpy="0 0 0" />-->
+        <origin xyz="0.0 0.0 0.0" rpy="0 0 0" />
         <parent link="${name}_link" />
         <child link="${name}_depth_frame"/>
@@ -47,5 +48,6 @@
       <link name="${name}_depth_optical_frame"/>
       <joint name="${name}_rgb_joint" type="fixed">
-        <origin xyz="0.0 0.022 0.0" rpy="0 0 0" />
+        <!--<origin xyz="0.0 0.022 0.0" rpy="0 0 0" />-->
+        <origin xyz="0.0 0.0 0.0" rpy="0 0 0" />
         <parent link="${name}_link" />
         <child link="${name}_rgb_frame"/>
@@ -70,5 +72,5 @@
             <horizontal_fov>${62.8 * M_PI/180.0}</horizontal_fov>
             <image>
-              <format>R8G8B8</format>
+              <format>B8G8R8</format>
               <width>640</width>
               <height>480</height>
