Commit message: Testing

File: single_lwr_example/single_lwr_robot/robot/single_lwr_robot.urdf.xacro (robot description, xacro)
@@ -3,4 +3,5 @@
 	<!-- Include all models -->
 	<xacro:include filename="$(find lwr_description)/model/kuka_lwr.urdf.xacro"/>
+	<link name="world" />
 	<!-- and assemble your robot -->
 	<link name="box">
@@ -14,16 +15,21 @@
 		</inertial>
 		<visual>
-			<origin xyz="0 0 0.50" rpy="0 0 0"/>
+			<origin xyz="0 0 2.05" rpy="0 0 0"/>
 			<geometry>
-				<box size="1.0 1.0 1.0"/>
+				<box size="2.0 0.1 0.1"/>
 			</geometry>
 		</visual>
 		<collision>
-			<origin xyz="0 0 0.50" rpy="0 0 0"/>
+			<origin xyz="0 0 2.05" rpy="0 0 0"/>
 			<geometry>
-				<box size="1.0 1.0 1.0"/>
+				<box size="2.0 0.1 0.1"/>
 			</geometry>
 		</collision>
 	</link>
+	<joint name="fix" type="fixed">
+		<origin xyz="0 0 0" rpy="0 0 0"/>
+		<parent link="world"/>
+		<child link="box"/>
+	</joint>
 	<gazebo reference="box">
 		<static>true</static>>
@@ -31,5 +37,5 @@
 	<!-- using the models -->
 	<xacro:kuka_lwr parent="box" name="lwr">
-		<origin xyz="0 0 1" rpy="0 0 0"/>
+		<origin xyz="0 0 2" rpy="0 3.14 0"/>
 	</xacro:kuka_lwr>
 </robot>

Commit message: Funzionante 0.0

File: single_lwr_example/single_lwr_robot/robot/single_lwr_robot.urdf.xacro (robot description, xacro)
@@ -39,4 +39,8 @@
 		<origin xyz="0 0 2" rpy="0 3.14 0"/>
 	</xacro:kuka_lwr>
-	<xacro:include filename="$(find lwr_testing)/sensors/asus_xtion_camera.urdf.xacro" />
+--
+	<xacro:include filename="$(find lwr_testing)/sensors/asus_camera.urdf.xacro" />
+	<xacro:asus_camera name="xtion" parent="lwr_7_link" >
+			<origin xyz="0 0 0" rpy="0 -1.57 0"/>
+	</xacro:asus_camera>
 </robot>

Commit message: Versione Funzionante con T_EE aggiustata

File: single_lwr_example/single_lwr_robot/robot/single_lwr_robot.urdf.xacro (robot description, xacro)
@@ -1,46 +1,73 @@
 <?xml version="1.0"?>
 <robot xmlns:xacro="http://www.ros.org/wiki/xacro" name="single_lwr_robot">
-	<!-- Include all models -->
-	<xacro:include filename="$(find lwr_description)/model/kuka_lwr.urdf.xacro"/>
-	<link name="world" />
-	<!-- and assemble your robot -->
-	<link name="box">
-		<inertial>
-			<mass value="5.0"/>
-			<origin rpy="0 0 0" xyz="0 0 0"/>
-			<inertia ixx="0.01"
-             iyy="0.01"
-             izz="0.01"
-             ixy="0" iyz="0" ixz="0"/>
-		</inertial>
-		<visual>
-			<origin xyz="0 0 2.05" rpy="0 0 0"/>
-			<geometry>
-				<box size="2.0 0.1 0.1"/>
-			</geometry>
-		</visual>
-		<collision>
-			<origin xyz="0 0 2.05" rpy="0 0 0"/>
-			<geometry>
-				<box size="2.0 0.1 0.1"/>
-			</geometry>
-		</collision>
-	</link>
-	<joint name="fix" type="fixed">
-		<origin xyz="0 0 0" rpy="0 0 0"/>
-		<parent link="world"/>
-		<child link="box"/>
-	</joint>
-	<gazebo reference="box">
-		<static>true</static>>
-	</gazebo>
-	<!-- using the models -->
-	<xacro:kuka_lwr parent="box" name="lwr">
-		<origin xyz="0 0 2" rpy="0 3.14 0"/>
-	</xacro:kuka_lwr>
---
-	<xacro:include filename="$(find lwr_testing)/sensors/asus_camera.urdf.xacro" />
-	<xacro:asus_camera name="xtion" parent="lwr_7_link" >
-			<origin xyz="0 0 0" rpy="0 -1.57 0"/>
-	</xacro:asus_camera>
+    <!-- Include all models -->
+    <xacro:include filename="$(find lwr_description)/model/kuka_lwr.urdf.xacro"/>
+    <link name="world" />
+    <!-- and assemble your robot -->
+    <link name="box">
+        <inertial>
+            <mass value="5.0"/>
+            <origin rpy="0 0 0" xyz="0 0 0"/>
+            <inertia ixx="0.01"
+                     iyy="0.01"
+                     izz="0.01"
+                     ixy="0" iyz="0" ixz="0"/>
+        </inertial>
+        <visual>
+            <origin xyz="0 0 2.05" rpy="0 0 0"/>
+            <geometry>
+                <box size="2.0 0.1 0.1"/>
+            </geometry>
+        </visual>
+        <collision>
+            <origin xyz="0 0 2.05" rpy="0 0 0"/>
+            <geometry>
+                <box size="2.0 0.1 0.1"/>
+            </geometry>
+        </collision>
+    </link>
+    <link name="table">
+        <inertial>
+            <mass value="5.0"/>
+            <origin rpy="0 0 0" xyz="0 0 0"/>
+            <inertia ixx="0.01"
+                     iyy="0.01"
+                     izz="0.01"
+                     ixy="0" iyz="0" ixz="0"/>
+        </inertial>
+        <visual>
+            <origin xyz="0 0 0.25" rpy="0 0 0"/>
+            <geometry>
+                <box size="0.5 0.5 0.5"/>
+            </geometry>
+        </visual>
+        <collision>
+            <origin xyz="0 0 0.25" rpy="0 0 0"/>
+            <geometry>
+                <box size="0.5 0.5 0.5"/>
+            </geometry>
+        </collision>
+    </link>
+    <joint name="fixt" type="fixed">
+        <origin xyz="0 0 0" rpy="0 0 0"/>
+        <parent link="world"/>
+        <child link="table"/>
+    </joint>
+    <joint name="fix" type="fixed">
+        <origin xyz="0 0 0" rpy="0 0 0"/>
+        <parent link="world"/>
+        <child link="box"/>
+    </joint>
+    <gazebo reference="box">
+        <static>true</static>>
+    </gazebo>
+    <!-- using the models -->
+    <xacro:kuka_lwr parent="box" name="lwr">
+        <origin xyz="0 0 2" rpy="0 3.14 0"/>
+    </xacro:kuka_lwr>
+    --
+    <xacro:include filename="$(find lwr_testing)/sensors/asus_camera.urdf.xacro" />
+    <xacro:asus_camera name="xtion" parent="lwr_7_link" >
+        <origin xyz="0 0 0" rpy="0 -1.57 0"/>
+    </xacro:asus_camera>
 </robot>
