Commit message: Super Prima Versione

File: lwr_description/model/kuka_lwr.gazebo.xacro (robot description, xacro)
@@ -1,42 +1,48 @@
 <?xml version="1.0"?>
 <robot xmlns:xacro="http://ros.org/wiki/xacro">
-	<xacro:macro name="kuka_lwr_gazebo" params="name">
-		<gazebo>
-			<plugin name="${name}_lwr_hw_sim" filename="liblwr_hw_gazebo_plugin.so">
-				<robotNamespace>${name}</robotNamespace>
-			</plugin>
-		</gazebo>
-		<gazebo reference="${name}_base_link">
-			<gravity>true</gravity>
-			<material>Gazebo/Orange</material>
-		</gazebo>
-		<gazebo reference="${name}_1_link">
-			<gravity>true</gravity>
-			<material>Gazebo/Orange</material>
-		</gazebo>
-		<gazebo reference="${name}_2_link">
-			<gravity>true</gravity>
-			<material>Gazebo/Orange</material>
-		</gazebo>
-		<gazebo reference="${name}_3_link">
-			<gravity>true</gravity>
-			<material>Gazebo/Orange</material>
-		</gazebo>
-		<gazebo reference="${name}_4_link">
-			<gravity>true</gravity>
-			<material>Gazebo/Orange</material>
-		</gazebo>
-		<gazebo reference="${name}_5_link">
-			<gravity>true</gravity>
-			<material>Gazebo/Orange</material>
-		</gazebo>
-		<gazebo reference="${name}_6_link">
-			<gravity>true</gravity>
-			<material>Gazebo/Orange</material>
-		</gazebo>
-		<gazebo reference="${name}_7_link">
-			<gravity>true</gravity>
-			<material>Gazebo/Grey</material>
-		</gazebo>
-	</xacro:macro>
+    <xacro:macro name="kuka_lwr_gazebo" params="name">
+        <gazebo>
+            <plugin name="${name}_lwr_hw_sim" filename="liblwr_hw_gazebo_plugin.so">
+                <robotNamespace>${name}</robotNamespace>
+            </plugin>
+        </gazebo>
+        <gazebo reference="${name}_base_link">
+            <gravity>true</gravity>
+            <material>Gazebo/Orange</material>
+        </gazebo>
+        <gazebo reference="${name}_1_link">
+            <gravity>true</gravity>
+            <material>Gazebo/Orange</material>
+        </gazebo>
+        <gazebo reference="${name}_2_link">
+            <gravity>true</gravity>
+            <material>Gazebo/Orange</material>
+        </gazebo>
+        <gazebo reference="${name}_3_link">
+            <gravity>true</gravity>
+            <material>Gazebo/Orange</material>
+        </gazebo>
+        <gazebo reference="${name}_4_link">
+            <gravity>true</gravity>
+            <material>Gazebo/Orange</material>
+        </gazebo>
+        <gazebo reference="${name}_5_link">
+            <gravity>true</gravity>
+            <material>Gazebo/Orange</material>
+        </gazebo>
+        <gazebo reference="${name}_6_link">
+            <gravity>true</gravity>
+            <material>Gazebo/Orange</material>
+        </gazebo>
+        <gazebo reference="${name}_7_link">
+            <gravity>true</gravity>
+            <material>Gazebo/Grey</material>
+        </gazebo>
+        <gazebo reference="table">
+            <mu1>1.2</mu1>
+            <mu2>1.2</mu2>
+            <gravity>false</gravity>
+            <material>Gazebo/Orange</material>
+        </gazebo>
+    </xacro:macro>
 </robot>

File: lwr_description/model/kuka_materials.xacro (robot description, xacro)
@@ -25,3 +25,6 @@
     <color rgba="0.0 0.0 0.8 1.0"/>
   </material>
+  <material name="Kuka/Brown">
+    <color rgba="0.9 0.7 0.0 1.0"/>
+  </material>
 </robot>

File: single_lwr_example/single_lwr_robot/robot/single_lwr_robot.urdf.xacro (robot description, xacro)
@@ -27,7 +27,7 @@
         </collision>
     </link>
-    <link name="table">
+   <!-- <link name="table">
         <inertial>
-            <mass value="5.0"/>
+            <mass value="5000.0"/>
             <origin rpy="0 0 0" xyz="0 0 0"/>
             <inertia ixx="0.01"
@@ -37,13 +37,13 @@
         </inertial>
         <visual>
-            <origin xyz="0 0 0.25" rpy="0 0 0"/>
+            <origin xyz="0 0 0.4" rpy="0 0 0"/>
             <geometry>
-                <box size="0.5 0.5 0.5"/>
+                <box size="1 1 0.8"/>
             </geometry>
         </visual>
         <collision>
-            <origin xyz="0 0 0.25" rpy="0 0 0"/>
+            <origin xyz="0 0 0.4" rpy="0 0 0"/>
             <geometry>
-                <box size="0.5 0.5 0.5"/>
+                <box size="1 1 0.8"/>
             </geometry>
         </collision>
@@ -53,5 +53,5 @@
         <parent link="world"/>
         <child link="table"/>
-    </joint>
+    </joint>-->
     <joint name="fix" type="fixed">
         <origin xyz="0 0 0" rpy="0 0 0"/>
